Commit message: feat: Add base_link description

File: urdf/simbot.xacro (robot description, xacro)
@@ -1,5 +1,4 @@
 <?xml version="1.0"?>
-<robot>
-	<xmlns:xacro="http://www.ros.org/wiki/xacro" name="simbot">
+<robot xmlns:xacro="http://www.ros.org/wiki/xacro" name="simbot">
 	<xacro:property name="base_width" value="0.16"/>
 	<xacro:property name="base_length" value="0.16"/>
@@ -11,5 +10,5 @@
 		<inertial>
 			<mass value="${m}"/>
-			<inertia>
+			<inertia
 				ixx="${m/12.0 * (d*d + h*h)}"
 				ixy="0.0"
@@ -17,6 +16,5 @@
 				iyy="${m/12.0 * (w*w + h*h)}"
 				iyz="0.0"
-				izz="${m/12.0 * (w*w + d*d)}"
-			</inertia>
+				izz="${m/12.0 * (w*w + d*d)}"/>
 		</inertial>
 	</xacro:macro>
@@ -30,3 +28,21 @@
 		</visual>
 	</link>
+	<link name="base_link">
+		<xacro:box_inertia m="10" w="${base_length}" h="${base_width}" d="0.01"/>
+		<visual>
+			<geometry>
+				<box size="${base_length} ${base_width} 0.01"/>
+			</geometry>
+		</visual>
+		<collision>
+			<geometry>
+				<box size="${base_length} ${base_width} 0.01"/>
+			</geometry>
+		</collision>
+	</link>
+	<joint name="base_link_joint" type="fixed">
+		<origin xyz="0 0 ${wheel_radius + 0.005}" rpy= "0 0 0"/>
+		<parent link="base_footprint"/>
+		<child link="base_link"/>
+	</joint>
 </robot>

Commit message: feat: Add wheel description

File: urdf/simbot.xacro (robot description, xacro)
@@ -46,3 +46,40 @@
 		<child link="base_link"/>
 	</joint>
+	<xacro:macro name="cylinder_inertial" params="m r h">
+		<inertial>
+			<mass value="${m}"/>
+			<inertia
+				ixx="${m*(3*r*r + h*h)/12}"
+				ixy="0"
+				ixz="0"
+				iyy="${m*(3*r*r + h*h)/12}"
+				iyz="0"
+				izz="${m*r*r/2}"/>
+		</inertial>
+	</xacro:macro>
+	<xacro:macro name="wheel" params="prefix reflect">
+		<link name="${prefix}_wheel">
+			<visual>
+				<origin xyz="0 0 0" rpy="${pi/2} 0 0"/>
+				<geometry>
+					<cylinder radius="${wheel_radius}" length="0.005"/>
+				</geometry>
+			</visual>
+			<collision>
+				<origin xyz="0 0 0" rpy="${pi/2} 0 0"/>
+				<geometry>
+					<cylinder radius="${wheel_radius}" length="0.005"/>
+				</geometry>
+			</collision>
+			<xacro:cylinder_inertial m="10" r="${wheel_radius}" h="0.005"/>
+		</link>
+		<joint name="${prefix}_wheel_joint" type="continuous">
+			<origin xyz="${wheel_joint_offset} ${(base_width/2 + base_wheel_gap) * reflect} -0.005" rpy="0 0 0"/>
+			<axis xyz="0 1 0" rpy="0 0 0"/>
+			<parent link="base_link"/>
+			<child link="${prefix}_wheel"/>
+		</joint>
+	</xacro:macro>
+	<xacro:wheel prefix="left" reflect="1"/>
+	<xacro:wheel prefix="right" reflect="-1"/>
 </robot>

Commit message: feat: Add caster wheel description

File: urdf/simbot.xacro (robot description, xacro)
@@ -7,4 +7,6 @@
 	<xacro:property name="wheel_seperation" value="0.15"/>
 	<xacro:property name="wheel_joint_offset" value="0.02"/>
+	<xacro:property name="caster_wheel_radius" value="${wheel_radius/2}"/>
+	<xacro:property name="caster_wheel_joint_offset" value="-0.052"/>
 	<xacro:macro name="box_inertia" params="m w h d">
 		<inertial>
@@ -83,3 +85,36 @@
 	<xacro:wheel prefix="left" reflect="1"/>
 	<xacro:wheel prefix="right" reflect="-1"/>
+	<xacro:macro name="sphere_inertia" params="m r">
+		<inertial>
+			<mass value="${m}"/>
+			<inertia
+				ixx="${2.0*m*r*r/5.0}"
+				ixy="0.0"
+				ixz="0.0"
+				iyy="${2.0*m*r*r/5.0}"
+				iyz="0.0"
+				izz="${2.0*m*r*r/5.0}"/>
+		</inertial>
+	</xacro:macro>
+	<link name="caster_wheel">
+		<visual>
+			<origin xyz="0 0 0" rpy="0 0 0"/>
+			<geometry>
+				<sphere radius="${caster_wheel_radius}"/>
+			</geometry>
+		</visual>
+		<collision>
+			<origin xyz="0 0 0" rpy="0 0 0"/>
+			<geometry>
+				<sphere radius="${caster_wheel_radius}"/>
+			</geometry>
+		</collision>
+		<xacro:sphere_inertia m="5" r="${caster_wheel_radius}"/>
+	</link>
+	<joint name="caster_wheel_joint" type="continuous">
+		<origin xyz="${caster_wheel_joint_offset} 0 -${caster_wheel_radius + 0.005}" rpy="0 0 0"/>
+		<axis xyz="0 1 0" rpy="0 0 0"/>
+		<parent link="base_link"/>
+		<child link="caster_wheel"/>
+	</joint>
 </robot>

Commit message: feat: Add material description

File: urdf/simbot.xacro (robot description, xacro)
@@ -1,4 +1,13 @@
 <?xml version="1.0"?>
 <robot xmlns:xacro="http://www.ros.org/wiki/xacro" name="simbot">
+	<material name="blue">
+		<color rgba="0 0 0.8 1"/>
+	</material>
+	<material name="black">
+		<color rgba="0 0 0 1"/>
+	</material>
+	<material name="white">
+		<color rgba="1 1 1 1"/>
+	</material>
 	<xacro:property name="base_width" value="0.16"/>
 	<xacro:property name="base_length" value="0.16"/>
@@ -36,4 +45,5 @@
 				<box size="${base_length} ${base_width} 0.01"/>
 			</geometry>
+			<material name="blue"/>
 		</visual>
 		<collision>
@@ -67,4 +77,5 @@
 					<cylinder radius="${wheel_radius}" length="0.005"/>
 				</geometry>
+				<material name="black"/>
 			</visual>
 			<collision>
@@ -103,4 +114,5 @@
 				<sphere radius="${caster_wheel_radius}"/>
 			</geometry>
+			<material name="white"/>
 		</visual>
 		<collision>

Commit message: feat: Add laser scanner description

File: urdf/simbot.xacro (robot description, xacro)
@@ -1,4 +1,7 @@
 <?xml version="1.0"?>
 <robot xmlns:xacro="http://www.ros.org/wiki/xacro" name="simbot">
+	<material name="red">
+		<color rgba="0.8 0 0 1"/>
+	</material>
 	<material name="blue">
 		<color rgba="0 0 0.8 1"/>
@@ -18,4 +21,10 @@
 	<xacro:property name="caster_wheel_radius" value="${wheel_radius/2}"/>
 	<xacro:property name="caster_wheel_joint_offset" value="-0.052"/>
+	<xacro:property name="laser_size_x" value="0.03"/>
+	<xacro:property name="laser_size_y" value="0.03"/>
+	<xacro:property name="laser_size_z" value="0.04"/>
+	<xacro:property name="laser_origin_x" value="0.065"/>
+	<xacro:property name="laser_origin_y" value="0"/>
+	<xacro:property name="laser_origin_z" value="0.035"/>
   <!--
   ==============================================================================
@@ -147,4 +156,28 @@
 	<!--
 	===============================================================================
+	Laser scanner
+	===============================================================================
+	-->
+	<link name="sensor_laser">
+		<visual>
+			<geometry>
+				<mesh filename="package://simbot_description/meshes/hokuyo.dae"/>
+			</geometry>
+			<material name="red"/>
+		</visual>
+		<collision>
+			<geometry>
+				<box size="${laser_size_x} ${laser_size_y} ${laser_size_z}"/>
+			</geometry>
+		</collision>
+		<xacro:box_inertia m="0.2" w="${laser_size_x}" h="${laser_size_y}" d="${laser_size_z}"/>
+	</link>
+	<joint name="sensor_laser_joint" type="fixed">
+		<origin xyz="${laser_origin_x} ${laser_origin_y} ${laser_origin_z}" rpy="0 0 0"/>
+		<parent link="base_link"/>
+		<child link="sensor_laser"/>
+	</joint>
+	<!--
+	===============================================================================
 	Gazebo plugins
 	===============================================================================
